Commit message: fixes for open/close hand

File: aero_shop/trx_s/urdf/trx_s.urdf.xacro (robot description, xacro)
@@ -143,5 +143,5 @@
     <origin xyz="0 ${0.028754 * reflect} -0.034615" rpy="0 -0 0 "/>
     <axis   xyz="1 0 0"/>
-    <limit lower="-3.14159" upper="3.14159" effort="100" velocity="0.5" />
+    <limit lower="-0.001" upper="0.001" effort="100" velocity="0.5" />
     <dynamics damping="0.2" friction="0" />
   </joint>
@@ -153,5 +153,5 @@
     <origin xyz="0 ${0.021716 * reflect} -0.013357" rpy="0 -0 0 "/>
     <axis   xyz="1 0 0"/>
-    <limit lower="-3.14159" upper="3.14159" effort="100" velocity="0.5" />
+    <limit lower="-0.001" upper="0.001" effort="100" velocity="0.5" />
     <dynamics damping="0.2" friction="0" />
   </joint>
