Commit message: overwrite limits for correct calculation

File: aero_shop/typeF_upperbody/urdf/aero_upper_typef.urdf.xacro (robot description, xacro)
@@ -466,5 +466,5 @@
     <axis   xyz="0 1 0"/>
     <!-- from -5 to 5 degrees-->
-    <limit lower="-0.087" upper="0.087" effort="100" velocity="0.9" />
+    <limit lower="-0.017" upper="0.017" effort="100" velocity="0.9" />
     <dynamics damping="0.2" friction="0" />
   </joint>
@@ -566,5 +566,5 @@
     <axis   xyz="0 1 0"/>
     <!-- from -5 to 5 degrees-->
-    <limit lower="-0.087" upper="0.087" effort="100" velocity="0.9" />
+    <limit lower="-0.017" upper="0.017" effort="100" velocity="0.9" />
     <dynamics damping="0.2" friction="0" />
   </joint>
